Commit message: valkyrie gravity compensation

File: ControlSystem/Valkyrie/Valkyrie_urdf/r5_urdf_rbdl.urdf (robot description, URDF)
Before this commit: robot valkyrie, 86 links, 85 joints
Links:
- removed link center_top_led_frame
- removed link leftHazardCamera_Frame
Joints:
- removed joint center_top_led_frame_joint
- removed joint leftHazardCamera_Offset
