Commit message: mercury assembly is done

File: Simulator/RobotModel/Mercury_Model/urdf/mercury.urdf (robot description, URDF)
Before this commit: robot mercury, 19 links, 18 joints
Links:
- link lfoot: geometry visual mesh filename=package://nao/meshes/meshes/V40/Updated_foot.dae scale=0.1 0.1 0.1
- link rfoot: geometry visual mesh filename=package://nao/meshes/meshes/V40/Updated_foot.dae scale=0.1 0.1 0.1
- link shank_l: geometry visual mesh filename=package://nao/meshes/meshes/V40/Updated_shin.dae scale=0.1 0.1 0.1
- link thigh_l: geometry visual mesh filename=package://nao/meshes/meshes/V40/Updated_thigh.dae scale=0.1 0.1 0.1
- link thigh_r: geometry visual mesh filename=package://nao/meshes/meshes/V40/Updated_thigh.dae scale=0.1 0.1 0.1
Joints:
- removed joint fixed_lfoot
- removed joint fixed_rfoot
- added joint ankle_l: type continuous, parent shank_l, child lfoot, origin xyz=0.0 0.0 -0.476 rpy=0 0 0, axis 0 1 0
- added joint ankle_r: type continuous, parent shank_r, child rfoot, origin xyz=0.0 0.0 -0.476 rpy=0 0 0, axis 0 1 0
