Commit message: mercury fixed in the air, joint position control

File: ControlSystem/Mercury/Mercury_urdf/mercury.urdf (robot description, URDF)
Before this commit: robot mercury, 19 links, 18 joints
Links:
- removed link torso
- added link body, mass 12.61; visual mesh filename=package://nao/meshes/meshes/V40/Updated_torso.dae scale=0.1 0.1 0.1
- link abduct_l: geometry visual mesh filename=package://nao/meshes/meshes/V40/abduction.dae scale=0.1 0.1 0.1
- link abduct_r: geometry visual mesh filename=package://nao/meshes/meshes/V40/abduction.dae scale=0.1 0.1 0.1
- link lfoot: geometry visual mesh filename=package://nao/meshes/meshes/V40/Updated_foot.dae scale=0.1 0.1 0.1
- link rfoot: geometry visual mesh filename=package://nao/meshes/meshes/V40/Updated_foot.dae scale=0.1 0.1 0.1
- link shank_l: geometry visual mesh filename=package://nao/meshes/meshes/V40/Updated_shin.dae scale=0.1 0.1 0.1
- link shank_r: geometry visual mesh filename=package://nao/meshes/meshes/V40/Updated_shin.dae scale=0.1 0.1 0.1
- link thigh_l: geometry visual mesh filename=package://nao/meshes/meshes/V40/Updated_thigh.dae scale=0.1 0.1 0.1
- link thigh_r: geometry visual mesh filename=package://nao/meshes/meshes/V40/Updated_thigh.dae scale=0.1 0.1 0.1
Joints:
- removed joint fixed_lfoot
- removed joint fixed_rfoot
- added joint ankle_l: type fixed, parent shank_l, child lfoot, origin xyz=0.0 0.0 -0.476 rpy=0 0 0, axis 0 1 0
- added joint ankle_r: type fixed, parent shank_r, child rfoot, origin xyz=0.0 0.0 -0.476 rpy=0 0 0, axis 0 1 0
- joint 1_torso_to_abduct_r_j: parent torso -> body
- joint 2_torso_to_abduct_l_j: parent torso -> body
- joint fixed_body_led3: parent torso -> body
- joint fixed_body_led4: parent torso -> body
- joint fixed_body_led5: parent torso -> body
- joint fixed_body_led6: parent torso -> body
- joint fixed_imu: parent torso -> body
- joint fixed_led0: parent torso -> body

File: Simulator/RobotModel/Mercury_Model/urdf/mercury.urdf (robot description, URDF)
Before this commit: robot mercury, 19 links, 18 joints
Links:
- removed link torso
- added link body, mass 12.61; visual mesh filename=package://nao/meshes/meshes/V40/Updated_torso.dae scale=0.1 0.1 0.1
- link lfoot: mass 0.000000000001 -> 0.123
- link rfoot: mass 0.000000000001 -> 0.123
Joints:
- joint 1_torso_to_abduct_r_j: parent torso -> body
- joint 2_torso_to_abduct_l_j: parent torso -> body
- joint fixed_body_led3: parent torso -> body
- joint fixed_body_led4: parent torso -> body
- joint fixed_body_led5: parent torso -> body
- joint fixed_body_led6: parent torso -> body
- joint fixed_imu: parent torso -> body
- joint fixed_led0: parent torso -> body

Commit message: mercury stand up test in progress

File: ControlSystem/Mercury/Mercury_urdf/mercury.urdf (robot description, URDF)
Before this commit: robot mercury, 19 links, 18 joints
Links:
- link body: mass 12.61 -> 8.9

File: Simulator/RobotModel/Mercury_Model/urdf/mercury.urdf (robot description, URDF)
Before this commit: robot mercury, 19 links, 18 joints
Links:
- link body: mass 12.61 -> 8.9

Commit message: reaction force transition data plot

File: ControlSystem/Mercury/Mercury_urdf/mercury.urdf (robot description, URDF)
Before this commit: robot mercury, 19 links, 18 joints
Links:
- link lfoot: mass 0.000000000001 -> 0.123
- link rfoot: mass 0.000000000001 -> 0.123
- link thigh_l: mass 3.0 -> 5.0
- link thigh_r: mass 3.0 -> 5.0

File: Simulator/RobotModel/Mercury_Model/urdf/mercury.urdf (robot description, URDF)
Before this commit: robot mercury, 19 links, 18 joints
Links:
- link thigh_l: mass 3.0 -> 5.0
- link thigh_r: mass 3.0 -> 5.0
